Commit message: Added body + wheels Works in Rviz

File: sim_tutorial/description/urdf/cybertruck.urdf.xacro (robot description, xacro)
@@ -2,19 +2,20 @@
 <robot name="cybertruck" xmlns:xacro="http://ros.org/wiki/xacro">
   <link name="base_link"/>
-  <!-- Your URDF code here -->
+  <!-- body link -->
   <link name="body_link">
     <visual>
         <origin xyz= "0 0 0" rpy = "0 0 0" />
-            <geometry>
-                <mesh filename="package://description/urdf/meshes/cybertruck_body.dae" />
-            </geometry>
+        <geometry>
+              <mesh filename="package://description/urdf/meshes/cybertruck_body.dae" />
+        </geometry>
     </visual>
     <collision>
         <origin xyz= "0 0 0" rpy = "0 0 0" />
-            <geometry>
-                <mesh filename="package://description/urdf/meshes/cybertruck_body.dae" />
+        <geometry>
+            <mesh filename="package://description/urdf/meshes/cybertruck_body.dae" />
         </geometry>
     </collision>
   </link>
+  <!-- body joint -->
   <joint name="body_joint" type="fixed">
     <parent link="base_link"/>
@@ -22,3 +23,5 @@
     <origin xyz = "0 0 0 " rpy="0 0 ${pi / 2}"/>
   </joint>
+  <!-- wheels -->
+  <xacro:include filename="$(find description)/urdf/wheels.urdf.xacro"/>
 </robot>

Commit message: Added body inertias, and roslaunch gazebo

File: sim_tutorial/description/urdf/cybertruck.urdf.xacro (robot description, xacro)
@@ -1,4 +1,7 @@
 <?xml version="1.0"?>
 <robot name="cybertruck" xmlns:xacro="http://ros.org/wiki/xacro">
+  <!-- Includes -->
+  <xacro:include filename="$(find description)/urdf/constants.xacro"/>
+  <xacro:include filename="$(find description)/urdf/inertias.xacro"/>
   <link name="base_link"/>
   <!-- body link -->
@@ -16,4 +19,7 @@
         </geometry>
     </collision>
+    <inertial>
+      <xacro:body_inertial m="${body_mass}" l="${body_length}" w="${body_width}" h="${body_height}" />
+    </inertial>
   </link>
   <!-- body joint -->

File: sim_tutorial/description/urdf/wheels.urdf.xacro (robot description, xacro)
@@ -20,4 +20,5 @@
     </link>
     <joint name="${fb}_${lr}_wheel_joint" type="continuous">
+        <!-- Wheel Link -->
         <parent link="body_link" />
         <child link="${fb}_${lr}_wheel_link"/>
